File: Kicad/PV-Monitor/PV-Monitor.kicad_pcb (KiCad board)
At the start: 2 copper layers, 29 parts, among them J1 Charge Controller, J2 Devices, U1 LM7805_TO220, U2 ACS758LCB-050B, U3 ACS758LCB-050B, U4 ACS758LCB-050B

Commit message: Update
Parts:
- added B1: ARDUINO_PRO_MINI, PV-Monitor:ARDUINO_PRO_MINI, F.Cu at (121.0, 67.5)
- moved C2 162.1 mm to (148.5, 70.0), turned to 180 degrees
- moved U1 140.5 mm to (154.5, 65.0), turned to 270 degrees
- moved C6 136.0 mm to (180.0, 86.0), turned to 90 degrees
- moved R2 128.0 mm to (137.5, 101.0)
- moved R7 127.1 mm to (175.5, 86.0), turned to 270 degrees
- moved R9 125.5 mm to (121.5, 86.0), turned to 270 degrees
- moved C7 123.4 mm to (153.0, 86.0), turned to 90 degrees
- moved R8 122.7 mm to (148.5, 86.0), turned to 270 degrees
- moved C9 122.3 mm to (166.5, 86.0), turned to 270 degrees
- moved R10 121.9 mm to (171.0, 86.0), turned to 270 degrees
- moved C1 119.3 mm to (148.5, 65.0), turned to 180 degrees
- moved C5 119.2 mm to (165.0, 92.0)
- moved C11 118.0 mm to (112.5, 86.0), turned to 270 degrees
- moved R5 110.9 mm to (137.5, 96.5)
- moved C10 102.8 mm to (139.0, 86.0), turned to 270 degrees
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Connections:
- C1 pad 1: Net-(C1-Pad1) -> /CHG_LOAD_POS
- U1 pad 1: Net-(C1-Pad1) -> /CHG_LOAD_POS
Routing:
- net GND: track 259.5 -> 624.6 mm, vias 0 -> 1
- net /5V: track 0.00 -> 179.1 mm, vias 0 -> 2
- net /CHG_LOAD_POS: track 103.7 -> 202.2 mm, vias 0 -> 3
- net /V_SENSE_LOAD: track 0.00 -> 82.1 mm, vias 0 -> 1
- net /V_SENSE_PV: track 0.00 -> 72.2 mm
- net /I_SENSE_PV: track 0.00 -> 63.1 mm, vias 0 -> 1
- net /V_SENSE_BATT: track 0.00 -> 60.8 mm, vias 0 -> 1
- net /I_SENSE_LOAD: track 0.00 -> 52.7 mm, vias 0 -> 1
- net /I_SENSE_BATT: track 0.00 -> 48.4 mm
- net /CHG_BATT_POS: track 79.0 -> 101.3 mm
- net /CHG_PV_POS: track 59.9 -> 77.6 mm
- net Net-(R9-Pad2): track 0.00 -> 5.09 mm
- net Net-(R8-Pad2): track 0.00 -> 5.01 mm
- net Net-(R7-Pad2): track 0.00 -> 4.95 mm

Commit message: Updates
Parts:
- added REF**: MountingHole_4.3mm_M4, MountingHole:MountingHole_4.3mm_M4, F.Cu at (201.0, 50.0)
- added REF**: MountingHole_4.3mm_M4, MountingHole:MountingHole_4.3mm_M4, F.Cu at (84.0, 50.0)
- added REF**: MountingHole_4.3mm_M4, MountingHole:MountingHole_4.3mm_M4, F.Cu at (84.0, 146.0)
- added REF**: MountingHole_4.3mm_M4, MountingHole:MountingHole_4.3mm_M4, F.Cu at (201.0, 146.0)
Routing:
- net GND: track 624.6 -> 633.6 mm
- added copper zone on F.Cu, net GND
Other:
- board outline added: 148 x 112 mm

Commit message: Updates
Parts:
- added D1: LED-3, LED:LED-1206, F.Cu at (172.6, 50.0)
- added D2: LED-4, LED:LED-1206, F.Cu at (176.0, 50.0)
- added D3: LED-1, LED:LED-1206, F.Cu at (165.7, 50.0)
- added D4: LED-2, LED:LED-1206, F.Cu at (169.2, 50.0)
- added JP1: Operation, Connector_PinHeader_2.54mm:PinHeader_1x03_P2.54mm_Vertical, F.Cu at (122.2, 50.0)
- added R13: 560, Resistor_SMD:R_1206_3216Metric_Pad1.42x1.75mm_HandSolder, F.Cu at (172.6, 56.8)
- added R14: 560, Resistor_SMD:R_1206_3216Metric_Pad1.42x1.75mm_HandSolder, F.Cu at (176.0, 56.8)
- added R15: 560, Resistor_SMD:R_1206_3216Metric_Pad1.42x1.75mm_HandSolder, F.Cu at (165.7, 56.8)
- added R16: 560, Resistor_SMD:R_1206_3216Metric_Pad1.42x1.75mm_HandSolder, F.Cu at (169.2, 56.8)
- added R17: 4k7, Resistor_SMD:R_1206_3216Metric_Pad1.42x1.75mm_HandSolder, F.Cu at (103.2, 50.0)
- added R18: 10k, Resistor_SMD:R_1206_3216Metric_Pad1.42x1.75mm_HandSolder, F.Cu at (128.2, 50.0)
- added R19: 10k, Resistor_SMD:R_1206_3216Metric_Pad1.42x1.75mm_HandSolder, F.Cu at (110.8, 50.0)
- added U5: DS18S20, Package_TO_SOT_THT:TO-92_Inline, F.Cu at (98.2, 51.2)
Connections:
- B1 pad 13: Net-(B1-Pad13) -> /LED_4
- B1 pad 14: Net-(B1-Pad14) -> /LED_3
- B1 pad 15: Net-(B1-Pad15) -> /LED_2
- B1 pad 16: Net-(B1-Pad16) -> /LED_1
- B1 pad 5: Net-(B1-Pad5) -> /DATA
- B1 pad 6: Net-(B1-Pad6) -> /SEL_2
- B1 pad 7: Net-(B1-Pad7) -> /SEL_1
Routing:
- net /SEL_2: track 0.00 -> 62.9 mm, vias 0 -> 1
- net /SEL_1: track 0.00 -> 62.4 mm, vias 0 -> 1
- net /DATA: track 0.00 -> 47.2 mm, vias 0 -> 2
- net /LED_4: track 0.00 -> 44.8 mm
- net /LED_3: track 0.00 -> 44.0 mm
- net /LED_2: track 0.00 -> 42.9 mm
- net /5V: track 179.1 -> 221.5 mm, vias 2 -> 3
- net /LED_1: track 0.00 -> 42.0 mm
- net GND: track 633.6 -> 616.7 mm
- net /I_SENSE_PV: track 63.1 -> 76.3 mm
- net /V_SENSE_BATT: track 60.8 -> 71.3 mm
- net /V_SENSE_PV: track 72.2 -> 68.3 mm
- net Net-(D4-PadA): track 0.00 -> 3.76 mm
- net Net-(D3-PadA): track 0.00 -> 3.76 mm
- net Net-(D2-PadA): track 0.00 -> 3.76 mm
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Other:
- board text added: "+"
- board text added: "-"
- board text added: "BATT"
- board text added: "LOAD"
- board text added: "PV"
- board text added: "PV Charger"
