File: Kicad/PV-Monitor/PV-Monitor.sch (KiCad schematic (older format))
At the start: 30 parts, among them J1 Charge Controller, J2 Devices, U1 LM7805_TO220, U2 ACS758LCB-050B, U3 ACS758LCB-050B, U4 ACS758LCB-050B

Commit message: Update
Parts:
- B1: footprint ARDUINO_PRO_MINI -> PV-Monitor:ARDUINO_PRO_MINI
Changed lines of the file:
@@
 F 0 "B1" H 3000 7110 45  0000 C CNN
 F 1 "ARDUINO_PRO_MINI" H 3000 7026 45  0000 C CNN
-F 2 "ARDUINO_PRO_MINI" H 3000 7000 20  0001 C CNN
+F 2 "PV-Monitor:ARDUINO_PRO_MINI" H 3000 7000 20  0001 C CNN
 F 3 "" H 3000 6050 50  0001 C CNN
 F 4 "XXX-00000" H 3000 6931 60  0000 C CNN "Field4"
@@
 DEV_LOAD_POS
 Wire Wire Line
-	1450 2950 1900 2950
+	1200 2950 1900 2950
 $EndSCHEMATC

Commit message: Updates
Parts:
- added D1: LED-3, LED:LED-1206, symbol SparkFun-LED:LED-GREEN1206
- added D2: LED-4, LED:LED-1206, symbol SparkFun-LED:LED-GREEN1206
- added D3: LED-1, LED:LED-1206, symbol SparkFun-LED:LED-GREEN1206
- added D4: LED-2, LED:LED-1206, symbol SparkFun-LED:LED-GREEN1206
- added JP1: Operation, Connector_PinHeader_2.54mm:PinHeader_1x03_P2.54mm_Vertical, symbol Jumper:Jumper_3_Open
- added R13, R14, R15, R16: 560, Resistor_SMD:R_1206_3216Metric_Pad1.42x1.75mm_HandSolder, symbol Device:R
- added R17: 4k7, Resistor_SMD:R_1206_3216Metric_Pad1.42x1.75mm_HandSolder, symbol Device:R
- added R18, R19: 10k, Resistor_SMD:R_1206_3216Metric_Pad1.42x1.75mm_HandSolder, symbol Device:R
- added U5: DS18S20, Package_TO_SOT_THT:TO-92_Inline, symbol Sensor_Temperature:DS18S20
Connections:
- net labels added: DATA, LED_1, LED_2, LED_3, LED_4, SEL_1, SEL_2
- wire segments 108 -> 148
Other:
- moved on the sheet: B1, C1, C2, J1, J2, U1

Commit message: Added initial software development
Parts:
- B1: symbol SparkFun-Boards:ARDUINO_PRO_MINI -> PV-Monitor-rescue:ARDUINO_PRO_MINI-SparkFun-Boards
- C1, C2: symbol SparkFun-Capacitors:1.0UF-1206-50V-10% -> PV-Monitor-rescue:1.0UF-1206-50V-10%-SparkFun-Capacitors
- D1, D2, D3, D4: symbol SparkFun-LED:LED-GREEN1206 -> PV-Monitor-rescue:LED-GREEN1206-SparkFun-LED
Connections:
- net labels added: 3V3
- wire segments 148 -> 149
Other:
- note added: "BUILTIN_LED"
Changed lines of the file:
@@
 LOAD-
 $Comp
-L SparkFun-PowerSymbols:GND #GND01
+L PV-Monitor-rescue:GND-SparkFun-PowerSymbols #GND01
 U 1 1 5FE8A971
 P 1850 1750
@@
 CHG_PV_POS
 $Comp
-L SparkFun-PowerSymbols:GND #GND05
+L PV-Monitor-rescue:GND-SparkFun-PowerSymbols #GND05
 U 1 1 5FE8B77B
 P 3950 1750
@@
 $EndComp
 $Comp
-L SparkFun-Capacitors:1.0UF-1206-50V-10% C1
+L PV-Monitor-rescue:1.0UF-1206-50V-10%-SparkFun-Capacitors C1
 U 1 1 5FE90E33
 P 2350 2750
@@
 $EndComp
 $Comp
-L SparkFun-Capacitors:1.0UF-1206-50V-10% C2
+L PV-Monitor-rescue:1.0UF-1206-50V-10%-SparkFun-Capacitors C2
 U 1 1 5FE916E0
 P 3450 2750
@@
 	3450 2850 3450 2950
 $Comp
-L SparkFun-PowerSymbols:GND #GND02
+L PV-Monitor-rescue:GND-SparkFun-PowerSymbols #GND02
 U 1 1 5FE94424
 P 2350 2950
@@
 $EndComp
 $Comp
-L SparkFun-PowerSymbols:GND #GND03
+L PV-Monitor-rescue:GND-SparkFun-PowerSymbols #GND03
 U 1 1 5FE94AB0
 P 2900 2950
@@
 $EndComp
 $Comp
-L SparkFun-PowerSymbols:GND #GND04
+L PV-Monitor-rescue:GND-SparkFun-PowerSymbols #GND04
 U 1 1 5FE94E09
 P 3450 2950
@@
 $EndComp
 $Comp
-L SparkFun-PowerSymbols:GND #GND06
+L PV-Monitor-rescue:GND-SparkFun-PowerSymbols #GND06
 U 1 1 5FEA2E3D
 P 6000 2350
@@
 $EndComp
 $Comp
-L SparkFun-PowerSymbols:GND #GND07
+L PV-Monitor-rescue:GND-SparkFun-PowerSymbols #GND07
 U 1 1 5FEA757D
 P 6000 4200
@@
 $EndComp
 $Comp
-L SparkFun-PowerSymbols:GND #GND08
+L PV-Monitor-rescue:GND-SparkFun-PowerSymbols #GND08
 U 1 1 5FEA8629
 P 6000 6050
@@
 $EndComp
 $Comp
-L SparkFun-PowerSymbols:GND #GND011
+L PV-Monitor-rescue:GND-SparkFun-PowerSymbols #GND011
 U 1 1 5FEAFC6C
 P 9350 2150
@@
 	9750 2050 9750 2150
 $Comp
-L SparkFun-PowerSymbols:GND #GND014
+L PV-Monitor-rescue:GND-SparkFun-PowerSymbols #GND014
 U 1 1 5FEB3BD2
 P 9750 2150
@@
 $EndComp
 $Comp
-L SparkFun-PowerSymbols:GND #GND010
+L PV-Monitor-rescue:GND-SparkFun-PowerSymbols #GND010
 U 1 1 5FEBFDE6
 P 9300 4000
@@
 	9700 3900 9700 4000
 $Comp
-L SparkFun-PowerSymbols:GND #GND013
+L PV-Monitor-rescue:GND-SparkFun-PowerSymbols #GND013
 U 1 1 5FEBFDF8
 P 9700 4000
@@
 $EndComp
 $Comp
-L SparkFun-PowerSymbols:GND #GND09
+L PV-Monitor-rescue:GND-SparkFun-PowerSymbols #GND09
 U 1 1 5FEC2405
 P 9250 5850
@@
 	9650 5750 9650 5850
 $Comp
-L SparkFun-PowerSymbols:GND #GND012
+L PV-Monitor-rescue:GND-SparkFun-PowerSymbols #GND012
 U 1 1 5FEC2417
 P 9650 5850
@@
 V_SENSE_PV
 $Comp
-L SparkFun-Boards:ARDUINO_PRO_MINI B1
+L PV-Monitor-rescue:ARDUINO_PRO_MINI-SparkFun-Boards B1
 U 1 1 5FEC493B
 P 2900 6650
@@
 $EndComp
 $Comp
-L SparkFun-PowerSymbols:GND #GND018
+L PV-Monitor-rescue:GND-SparkFun-PowerSymbols #GND018
 U 1 1 5FEE0023
 P 7050 2350
@@
 $EndComp
 $Comp
-L SparkFun-PowerSymbols:GND #GND019
+L PV-Monitor-rescue:GND-SparkFun-PowerSymbols #GND019
 U 1 1 5FEE4391
 P 7050 4200
@@
 $EndComp
 $Comp
-L SparkFun-PowerSymbols:GND #GND020
+L PV-Monitor-rescue:GND-SparkFun-PowerSymbols #GND020
 U 1 1 5FEE7784
 P 7050 6050
@@
 	6550 5950 6550 6050
 $Comp
-L SparkFun-PowerSymbols:GND #GND017
+L PV-Monitor-rescue:GND-SparkFun-PowerSymbols #GND017
 U 1 1 5FF0581C
 P 6550 6050
@@
 	7400 5950 7400 6050
 $Comp
-L SparkFun-PowerSymbols:GND #GND023
+L PV-Monitor-rescue:GND-SparkFun-PowerSymbols #GND023
 U 1 1 5FF07F7A
 P 7400 6050
@@
 	6550 4100 6550 4200
 $Comp
-L SparkFun-PowerSymbols:GND #GND016
+L PV-Monitor-rescue:GND-SparkFun-PowerSymbols #GND016
 U 1 1 5FF0AA2B
 P 6550 4200
@@
 	7400 4100 7400 4200
 $Comp
-L SparkFun-PowerSymbols:GND #GND022
+L PV-Monitor-rescue:GND-SparkFun-PowerSymbols #GND022
 U 1 1 5FF0D484
 P 7400 4200
@@
 	7400 2250 7400 2350
 $Comp
-L SparkFun-PowerSymbols:GND #GND021
+L PV-Monitor-rescue:GND-SparkFun-PowerSymbols #GND021
 U 1 1 5FF0FCE7
 P 7400 2350
@@
 	6550 2250 6550 2350
 $Comp
-L SparkFun-PowerSymbols:GND #GND015
+L PV-Monitor-rescue:GND-SparkFun-PowerSymbols #GND015
 U 1 1 5FF12438
 P 6550 2350
@@
 $EndComp
 $Comp
-L SparkFun-PowerSymbols:GND #GND025
+L PV-Monitor-rescue:GND-SparkFun-PowerSymbols #GND025
 U 1 1 5FEA8B62
 P 5350 7400
@@
 	3350 6950 4050 6950
 Wire Wire Line
-	3350 7050 4050 7050
-$Comp
-L SparkFun-LED:LED-GREEN1206 D4
+	1900 6650 2450 6650
+$Comp
+L PV-Monitor-rescue:LED-GREEN1206-SparkFun-LED D4
 U 1 1 5FEE1190
 P 3400 4150
@@
 $EndComp
 $Comp
-L SparkFun-LED:LED-GREEN1206 D3
+L PV-Monitor-rescue:LED-GREEN1206-SparkFun-LED D3
 U 1 1 5FEE2AEA
 P 3400 3600
@@
 $EndComp
 $Comp
-L SparkFun-LED:LED-GREEN1206 D1
+L PV-Monitor-rescue:LED-GREEN1206-SparkFun-LED D1
 U 1 1 5FEE3325
 P 2500 3600
@@
 $EndComp
 $Comp
-L SparkFun-LED:LED-GREEN1206 D2
+L PV-Monitor-rescue:LED-GREEN1206-SparkFun-LED D2
 U 1 1 5FEE39DA
 P 2500 4150
@@
 	2950 4150 2950 4300
 $Comp
-L SparkFun-PowerSymbols:GND #GND024
+L PV-Monitor-rescue:GND-SparkFun-PowerSymbols #GND024
 U 1 1 5FF4BCCD
 P 2950 4300
@@
 Text Label 3450 6950 0    50   ~ 0
 LED_3
-Text Label 3450 7050 0    50   ~ 0
+Text Label 1900 6650 0    50   ~ 0
 LED_4
 Text Label 4200 3600 0    50   ~ 0
@@
 	2950 5150 2950 5200
 $Comp
-L SparkFun-PowerSymbols:GND #GND026
+L PV-Monitor-rescue:GND-SparkFun-PowerSymbols #GND026
 U 1 1 5FFB8EBF
 P 2950 5200
@@
 $EndComp
 Text Label 4000 5000 0    50   ~ 0
-5V
+3V3
 Text Label 3900 4750 0    50   ~ 0
 SEL_1
@@
 SEL_2
 Text Label 1700 5000 0    50   ~ 0
-5V
+3V3
 Wire Wire Line
 	2450 6450 1900 6450
@@
 Text Label 1900 6550 0    50   ~ 0
 SEL_1
+Wire Wire Line
+	3350 6250 4050 6250
+Text Label 3450 6250 0    50   ~ 0
+3V3
+Text Notes 3450 7050 0    50   ~ 0
+BUILTIN_LED
 $EndSCHEMATC
